Commit message: Some simple simulations

File: models/furuta.urdf (robot description, URDF)
Before this commit: robot furuta_pendulum, 3 links, 2 joints
Links:
- link arm_link: geometry visual cylinder length=0.2 radius=0.01
- link base_link: mass 1.0 -> None; geometry visual cylinder length=0.05 radius=0.05
- link pendulum_link: geometry visual cylinder length=0.2 radius=0.008
Joints:
- joint arm_joint: origin (none) -> xyz=0 0 0.05
